File: tests/regression/schematics/hierarchical/hierarchical.kicad_sch (KiCad schematic)
At the start: 1 part

Commit message: kicad test cases
Parts:
- R1: symbol (none) -> Device:R
Connections:
- net PowerBuffer/SIGNAL: now also R1.2
- net VCC: now also R1.1
Changed lines of the file:
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@@
   (generator kicad_condenser_test)
   ; R1 at (10, 10):  pin2 abs=(10,8.984)=VCC  pin1 abs=(10,11.016)=SIGNAL
-  (symbol "Device:R" (at 10 10 0) (unit 1) (in_bom yes) (on_board yes)
-    (property "Reference" "R1" (id 0) (at 10 10 0))
-    (property "Value" "4k7" (id 1) (at 10 10 0))
-    (property "Footprint" "Resistor_SMD:R_0402" (id 2) (at 10 10 0))
-    (property "Datasheet" "~" (id 3) (at 10 10 0))
+  (symbol
+    (lib_id "Device:R")
+    (at 10 10 0)
+    (unit 1)
+    (in_bom yes)
+    (on_board yes)
+    (property "Reference" "R1" (at 10 10 0))
+    (property "Value" "4k7" (at 10 10 0))
+    (property "Footprint" "Resistor_SMD:R_0402" (at 10 10 0))
+    (property "Datasheet" "~" (at 10 10 0))
     (instances
       (project "hierarchical"
