File: tests/regression/schematics/hierarchical/sub.kicad_sch (KiCad schematic)
At the start: 1 part

Commit message: kicad test cases
Parts:
- C1: symbol (none) -> Device:C
Connections:
- net GND: now also C1.2
- net SIGNAL: now also C1.1
Changed lines of the file:
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@@
   (hierarchical_label "SIGNAL" (shape input) (at 10 5 0))
   ; C1 at (10, 12):  pin2 abs=(10,10.984)=SIGNAL  pin1 abs=(10,13.016)=GND
-  (symbol "Device:C" (at 10 12 0) (unit 1) (in_bom yes) (on_board yes)
-    (property "Reference" "C1" (id 0) (at 10 12 0))
-    (property "Value" "100n" (id 1) (at 10 12 0))
-    (property "Footprint" "Capacitor_SMD:C_0402" (id 2) (at 10 12 0))
-    (property "Datasheet" "~" (id 3) (at 10 12 0))
+  (symbol
+    (lib_id "Device:C")
+    (at 10 12 0)
+    (unit 1)
+    (in_bom yes)
+    (on_board yes)
+    (property "Reference" "C1" (at 10 12 0))
+    (property "Value" "100n" (at 10 12 0))
+    (property "Footprint" "Capacitor_SMD:C_0402" (at 10 12 0))
+    (property "Datasheet" "~" (at 10 12 0))
     (instances
       (project "hierarchical"
